File: glow/glow.kicad_sch (KiCad schematic)
At the start: 36 parts, among them J3 In, J5 Out

Commit message: routing
Parts:
- added H1, H2: M4, MountingHole:MountingHole_4mm_Pad_Via, symbol Mechanical:MountingHole_Pad
Connections:
- new net GND: H1.1, H2.1
Changed lines of the file:
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@@
     (pin "4")
+  )
+  (symbol (lib_id "Mechanical:MountingHole_Pad") (at 88.9 33.02 0) (unit 1)
+    (in_bom yes) (on_board yes)
+    (property "Reference" "H2" (id 0) (at 87.63 27.94 0)
+      (effects (font (size 1.27 1.27)) (justify left))
+    )
+    (property "Value" "M4" (id 1) (at 87.63 45.212 0)
+      (effects (font (size 1.27 1.27)) (justify left))
+    )
+    (property "Footprint" "MountingHole:MountingHole_4mm_Pad_Via" (id 2) (at 88.9 33.02 0)
+      (effects (font (size 1.27 1.27)) hide)
+    )
+    (property "Datasheet" "~" (id 3) (at 88.9 33.02 0)
+      (effects (font (size 1.27 1.27)) hide)
+    )
+    (pin "1")
   )
   (symbol (lib_id "LED:SK6812MINI") (at 274.32 90.805 0) (unit 1)
@@
     (pin "3")
     (pin "4")
+  )
+  (symbol (lib_id "Mechanical:MountingHole_Pad") (at 82.55 33.02 0) (unit 1)
+    (in_bom yes) (on_board yes)
+    (property "Reference" "H1" (id 0) (at 81.28 27.94 0)
+      (effects (font (size 1.27 1.27)) (justify left))
+    )
+    (property "Value" "M4" (id 1) (at 81.28 45.212 0)
+      (effects (font (size 1.27 1.27)) (justify left))
+    )
+    (property "Footprint" "MountingHole:MountingHole_4mm_Pad_Via" (id 2) (at 82.55 33.02 0)
+      (effects (font (size 1.27 1.27)) hide)
+    )
+    (property "Datasheet" "~" (id 3) (at 82.55 33.02 0)
+      (effects (font (size 1.27 1.27)) hide)
+    )
+    (pin "1")
   )
   (symbol (lib_id "Connector:Conn_01x03_Female") (at 32.8422 40.005 0) (unit 1)
@@
     (pin "4")
   )
+  (symbol (lib_id "power:GND") (at 88.9 35.56 0) (unit 1)
+    (in_bom yes) (on_board yes)
+    (property "Reference" "#PWR0102" (id 0) (at 88.9 41.91 0)
+      (effects (font (size 1.27 1.27)) hide)
+    )
+    (property "Value" "GND" (id 1) (at 88.744 42.5449 90)
+      (effects (font (size 1.27 1.27)) (justify left))
+    )
+    (property "Footprint" "" (id 2) (at 88.9 35.56 0)
+      (effects (font (size 1.27 1.27)) hide)
+    )
+    (property "Datasheet" "" (id 3) (at 88.9 35.56 0)
+      (effects (font (size 1.27 1.27)) hide)
+    )
+    (pin "1")
+  )
   (symbol (lib_id "LED:SK6812MINI") (at 186.182 69.85 0) (unit 1)
     (in_bom yes) (on_board yes)
@@
     (pin "3")
     (pin "4")
+  )
+  (symbol (lib_id "power:GND") (at 82.55 35.56 0) (unit 1)
+    (in_bom yes) (on_board yes)
+    (property "Reference" "#PWR0101" (id 0) (at 82.55 41.91 0)
+      (effects (font (size 1.27 1.27)) hide)
+    )
+    (property "Value" "GND" (id 1) (at 82.394 42.5449 90)
+      (effects (font (size 1.27 1.27)) (justify left))
+    )
+    (property "Footprint" "" (id 2) (at 82.55 35.56 0)
+      (effects (font (size 1.27 1.27)) hide)
+    )
+    (property "Datasheet" "" (id 3) (at 82.55 35.56 0)
+      (effects (font (size 1.27 1.27)) hide)
+    )
+    (pin "1")
   )
   (symbol (lib_id "LED:SK6812MINI") (at 208.407 90.805 0) (unit 1)
@@
   )
   (symbol_instances
+    (path "/d681d8bf-5312-43f2-9d28-55d47254dd88"
+      (reference "#PWR0101") (unit 1) (value "GND") (footprint "")
+    )
+    (path "/b3fe7ca7-68d6-482a-8ea0-c1f1e489c7f2"
+      (reference "#PWR0102") (unit 1) (value "GND") (footprint "")
+    )
     (path "/03921f2e-45fd-46df-ac7a-a595d622cae4"
       (reference "C1") (unit 1) (value "C") (footprint "Capacitor_SMD:C_1206_3216Metric_Pad1.42x1.75mm_HandSolder")
@@
       (reference "D60") (unit 1) (value "SK6812MINI") (footprint "libs2:YS-SK6812MINI-E_REVERSE_NO_EDGECUT")
     )
+    (path "/86b3ecc5-4919-498e-a5fc-2c1b3a23f15b"
+      (reference "H1") (unit 1) (value "M4") (footprint "MountingHole:MountingHole_4mm_Pad_Via")
+    )
+    (path "/36e4075f-5169-42a6-8463-6ac1b4fe40b4"
+      (reference "H2") (unit 1) (value "M4") (footprint "MountingHole:MountingHole_4mm_Pad_Via")
+    )
     (path "/86e9b100-0cb2-4e0a-bfe5-e176a6ebe6f5"

Commit message: routing, logos
Connections:
- net Gnd: now also D21.2 (VSS), D22.2 (VSS), D23.2 (VSS), D24.2 (VSS), D25.2 (VSS), D26.2 (VSS), D37.2 (VSS), D38.2 (VSS), D39.2 (VSS), D40.2 (VSS), D41.2 (VSS), D42.2 (VSS), D47.2 (VSS), D48.2 (VSS), D49.2 (VSS), D50.2 (VSS), D51.2 (VSS), D52.2 (VSS), D55.2 (VSS), D56.2 (VSS), D57.2 (VSS), D58.2 (VSS), D59.2 (VSS), D60.2 (VSS)
- net Vcc: now also D21.4 (VDD), D22.4 (VDD), D23.4 (VDD), D24.4 (VDD), D25.4 (VDD), D26.4 (VDD), D33.4 (VDD), D37.4 (VDD), D38.4 (VDD), D39.4 (VDD), D40.4 (VDD), D41.4 (VDD), D42.4 (VDD), D47.4 (VDD), D48.4 (VDD), D49.4 (VDD), D5.4 (VDD), D50.4 (VDD), D51.4 (VDD), D52.4 (VDD), D55.4 (VDD), D56.4 (VDD), D57.4 (VDD), D58.4 (VDD), D59.4 (VDD), D60.4 (VDD), D7.4 (VDD)
- net at D21.3 (DIN), D22.3 (DIN), D33.1 (DOUT): now also D34.1 (DOUT)
- net at D42.1 (DOUT), D48.3 (DIN): now also D41.1 (DOUT), D47.3 (DIN)
- net at D5.3 (DIN), D6.3 (DIN): now also R1.2, R2.2
